File: trialkb.kicad_pcb (KiCad board)
At the start: 2 copper layers, 36.5 x 38.1 mm, 24 parts, among them SW1 SW_Push, U1 ATmega32U4-AU, Y1 16MHz

Commit message: routing complete
Parts:
- SW1: footprint random-keyboard-parts:Reset_Pretty -> random-keyboard-parts:SKQG-1155865; moved to B.Cu
- moved R2 173.6 mm to (32.5, 57.3), turned to 90 degrees
- moved R1 165.4 mm to (29.4, 57.3), turned to 90 degrees
- moved SW1 151.3 mm to (31.0, 75.4)
- moved F1 146.3 mm to (28.6, 65.1), turned to 90 degrees
- moved R3 145.9 mm to (37.3, 55.7), turned to 270 degrees
- moved R4 28.7 mm to (61.1, 72.3)
- moved C6 7.32 mm to (41.3, 72.2), turned to 270 degrees
- moved C7 1.12 mm to (40.6, 65.9)
- moved C1 0.64 mm to (57.0, 77.0)
Connections:
- U1 pad 27: Net-(U1-Pad27) -> ROW0
- U1 pad 28: Net-(U1-Pad28) -> COL1
- U1 pad 29: Net-(U1-Pad29) -> COL0
- U1 pad 30: Net-(U1-Pad30) -> ROW1
Routing:
- net GND: track 0.00 -> 132.4 mm
- net +5V: track 0.00 -> 101.5 mm, vias 0 -> 5
- net COL1: track 0.00 -> 52.3 mm
- net ROW1: track 0.00 -> 51.3 mm
- net Net-(R3-Pad2): track 0.00 -> 48.9 mm, vias 0 -> 2
- net ROW0: track 0.00 -> 47.6 mm
- net COL0: track 0.00 -> 35.6 mm
- net Net-(R1-Pad1): track 0.00 -> 23.7 mm
- net Net-(R2-Pad1): track 0.00 -> 22.2 mm
- net Net-(C5-Pad1): track 0.00 -> 14.2 mm
- net Net-(C4-Pad1): track 0.00 -> 9.94 mm
- net Net-(D4-Pad2): track 0.00 -> 6.62 mm
- net Net-(D2-Pad2): track 0.00 -> 6.62 mm
- net Net-(D3-Pad2): track 0.00 -> 6.62 mm
- net Net-(D1-Pad2): track 0.00 -> 6.62 mm
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Other:
- board size 36.5 x 38.1 mm -> 77 x 38.1 mm
- net class Default: trace_width 0.25 -> 0.254
- net class Power added: clearance 0.2, trace_width 0.254, via_dia 0.8, via_drill 0.4

Commit message: ready for production
Parts:
- moved C5 8.74 mm to (46.8, 53.0), turned to 270 degrees
- moved C4 7.94 mm to (54.8, 53.0), turned to 90 degrees
- turned SW1 to 180 degrees
Routing:
- net GND: track 132.4 -> 150.5 mm
- net Net-(R3-Pad2): track 48.9 -> 33.1 mm
- net VCC: track 0.00 -> 12.3 mm
- added copper zone on B.Cu, net GND
Other:
- board text added: "nvmnd - trialkb"
